Commit message: update

File: urdf/srobot.urdf (robot description, URDF)
Before this commit: robot srobot, 4 links, 3 joints
Links:
- removed link imu_frame
- link base_link: mass 33.2741044624964 -> 36.2523043272947
- link base_scan: mass 0.204546095137456 -> 0.204546095121516
- link imu_link: mass 0.0150303013778878 -> 0.0150303013778881
Joints:
- removed joint imuframe_joint
- joint imu_joint: origin xyz=0.1265 0 0.0807 rpy=0 0 1.5708 -> xyz=-0.042 0 0.5387 rpy=0 0 -1.5708
- joint scan_joint: origin xyz=0.1435 -0.001 -0.0109 rpy=3.1416 0 0 -> xyz=0.1755 0 0.10075 rpy=2.1649E-15 1.2228E-17 -4.2633E-16
